File: OrbitX-PCB/Orbit.kicad_pcb (KiCad board)
At the start: 2 copper layers, 261.9 x 117.5 mm, 165 parts, among them J1 PJ-3200B-4A, J11 PJ-3200B-4A, J12 AVR-ISP-6, J13 Breakaway_Tabs, J14 Breakaway_Tabs, J17 Breakaway_Tabs, J18 Breakaway_Tabs, J19 Breakaway_Tabs, J2 AVR-ISP-6, J3 Breakaway_Tabs, J5 Breakaway_Tabs, J6 Breakaway_Tabs, J7 Breakaway_Tabs, J9 Breakaway_Tabs, SW1 SW_Push, SW2 SW_Push, U1 ATmega32U4-MU, U2 PRTR5V0U2X, U3 ATmega32U4-MU, U4 PRTR5V0U2X, Y1 16MHz, Y2 16MHz

Commit message: Build new OrbitX PCB
Parts:
- removed the G*** at (288.9, 130.2)
- removed the G*** at (52.4, 95.2)
- removed the G*** at (43.7, 130.2)
- removed the G*** at (144.5, 118.3) (x2)
- removed the G*** at (181.0, 118.3) (x2)
- removed the G*** at (272.3, 95.2)
- removed the G*** at (51.6, 95.2)
- removed the G*** at (273.1, 95.2)
- removed J12, J2: AVR-ISP-6, random-keyboard-parts:Reset_Pretty-Mask
- added C15: 0.1uF, Capacitor_SMD:C_0603_1608Metric, B.Cu at (84.9, 101.6)
- added C16: 0.1uF, Capacitor_SMD:C_0603_1608Metric, B.Cu at (188.9, 84.9)
- added G***: LOGO, locallib:ai-ring-6mm-Combined, B.Cu at (164.3, 119.9)
- added G***: LOGO, locallib:ai-ring-6mm-Combined, B.Cu at (128.6, 119.9)
- added G***: LOGO, locallib:ai-ring-6mm-Combined, F.Cu at (259.6, 104.8)
- added G***: LOGO, locallib:ai-ring-6mm-Combined, F.Cu at (33.3, 104.8)
- added G***: LOGO, locallib:orbitx, B.Cu at (33.3, 94.5)
- added G***: LOGO, locallib:orbitx, F.Cu at (33.3, 95.2)
- added G***: LOGO, locallib:orbitx, B.Cu at (259.6, 94.5)
- added G***: LOGO, locallib:orbitx, F.Cu at (259.6, 95.2)
- added REF**: orbitx-outline, locallib:orbitx-outline, F.Cu at (23.8, 47.6)
- J13, J14, J17, J18, J19, J3, J5, J6, J7, J9: moved to F.Cu
- MX1, MX10, MX11, MX13, MX14, MX15, MX16, MX17, MX18, MX19, MX2, MX20, MX21, MX22, MX23, MX24, MX25, MX26, MX27, MX28, MX29, MX3, MX30, MX31, MX32, MX33, MX34, MX35, MX36, MX37, MX38, MX39, MX4, MX41, MX42, MX43, MX44, MX45, MX46, MX47, MX48, MX5, MX6, MX7, MX8, MX9: footprint MX_Alps_Hybrid:MX-1U-NoLED -> MX_Only:MXOnly-1U-NoLED
- MX12, MX40: footprint MX_Alps_Hybrid:MX-1.5U-NoLED -> MX_Only:MXOnly-1.5U-NoLED
- U1, U3: value ATmega32U4-MU -> ATmega32U4-AU; footprint Package_DFN_QFN:QFN-44-1EP_7x7mm_P0.5mm_EP5.2x5.2mm -> Package_QFP:TQFP-44_10x10mm_P0.8mm
- moved FID1 273.8 mm to (17.5, 18.3)
- moved FID3 241.3 mm to (275.4, 137.3), turned to 180 degrees
- moved FID2 241.3 mm to (275.4, 18.3)
- moved J3 228.5 mm to (33.3, 114.0)
- moved J17 198.2 mm to (259.6, 114.0)
- moved J18 195.3 mm to (81.0, 106.9), turned to 0 degrees
- moved J6 151.0 mm to (100.0, 33.5)
- moved J13 120.0 mm to (211.9, 106.9)
- moved J14 115.4 mm to (211.9, 114.0), turned to 0 degrees
- moved J5 86.5 mm to (61.9, 33.5)
- moved J9 72.1 mm to (231.0, 33.5)
- moved R41 36.4 mm to (71.4, 94.5), turned to 180 degrees
- moved R9 36.1 mm to (83.3, 82.5)
- moved R42 35.1 mm to (71.4, 96.8), turned to 180 degrees
- moved J19 31.8 mm to (81.0, 114.0), turned to 0 degrees
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Connections:
- C14 pad 1: +5VA -> VDC
- C7 pad 1: +5V -> VBUS
- U1 pad 1: Net-(U1-Pad1) -> COL0
- U1 pad 10: MOSI -> Net-(U1-Pad10)
- U1 pad 11: MISO -> Net-(U1-Pad11)
- U1 pad 25: Net-(U1-Pad25) -> ROW2
- U1 pad 26: Net-(U1-Pad26) -> ROW1
- U1 pad 27: Net-(U1-Pad27) -> ROW0
- U1 pad 28: ROW0 -> Net-(U1-Pad28)
- U1 pad 29: ROW1 -> Net-(U1-Pad29)
- U1 pad 30: ROW2 -> Net-(U1-Pad30)
- U1 pad 36: ROW3 -> Net-(U1-Pad36)
- U1 pad 37: Net-(U1-Pad37) -> COL1
- U1 pad 38: COL3 -> Net-(U1-Pad38)
- U1 pad 39: COL2 -> Net-(U1-Pad39)
- U1 pad 40: COL1 -> Net-(U1-Pad40)
- U1 pad 41: COL0 -> ROW3
- U1 pad 8: Net-(U1-Pad8) -> COL3
- U1 pad 9: SCK -> COL2
- U3 pad 1: COL2-R -> Net-(U3-Pad1)
- U3 pad 10: MOSI-R -> COL5-R
- U3 pad 11: MISO-R -> COL4-R
- U3 pad 26: ROW1-R -> COL0-R
- U3 pad 27: ROW0-R -> ROW1-R
- U3 pad 28: Net-(U3-Pad28) -> ROW2-R
- U3 pad 29: Net-(U3-Pad29) -> ROW0-R
- U3 pad 30: Net-(U3-Pad30) -> COL1-R
- U3 pad 31: COL0-R -> Net-(U3-Pad31)
- U3 pad 32: COL1-R -> Net-(U3-Pad32)
- U3 pad 36: ROW2-R -> Net-(U3-Pad36)
- U3 pad 39: COL5-R -> Net-(U3-Pad39)
- U3 pad 40: COL4-R -> Net-(U3-Pad40)
- U3 pad 41: COL3-R -> Net-(U3-Pad41)
- U3 pad 8: Net-(U3-Pad8) -> COL3-R
- U3 pad 9: SCK-R -> COL2-R
Routing:
- net ROW3-R: track 172.7 -> 106.1 mm, vias 7 -> 2
- net RESET: track 42.6 -> 87.4 mm, vias 4 -> 6
- net MISO-R: track 34.7 -> 0.00 mm
- net GNDA: track 281.7 -> 310.0 mm, vias 6 -> 4
- net SCK-R: track 27.2 -> 0.00 mm
- net MOSI: track 25.3 -> 0.00 mm, vias 1 -> 0
- net ROW2-R: track 88.0 -> 112.6 mm
- net MOSI-R: track 23.9 -> 0.00 mm
- net SCK: track 22.7 -> 0.00 mm, vias 1 -> 0
- net MISO: track 22.5 -> 0.00 mm, vias 1 -> 0
- net +5V: track 173.6 -> 151.5 mm, vias 11 -> 7
- net COL3: track 90.1 -> 69.6 mm, vias 4 -> 0
- net COL3-R: track 105.1 -> 84.5 mm
- net RESET-R: track 57.2 -> 39.3 mm, vias 3 -> 2
- net COL4-R: track 131.2 -> 113.8 mm, vias 3 -> 1
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Other:
- board size 261.9 x 117.5 mm -> 263.8 x 125 mm
- board text removed: "PCB Rev 1.0 20190625 | kb.ai03.me"
- board text removed: "PCB Rev 1.0 | 20190625"
- board text removed: "by ai03"

Commit message: Finalize decal
Parts:
- added G***: LOGO, locallib:orbitx, F.Cu at (26.2, 135.7)
Other:
- board text added: "Compact Ergonomic Keyboard by ai03"
- board text added: "PCB Revision 2.0 20190930"
- board text added: "R2.0 20190930"
