File: Orbit-PCB/Orbit.kicad_pcb (KiCad board)
At the start: 2 copper layers, 303.2 x 145.3 mm, 301 parts, among them J1 PJ-3200B-4A, J10 Breakaway_Tabs, J11 PJ-3200B-4A, J12 AVR-ISP-6, J13 Breakaway_Tabs, J14 Breakaway_Tabs, J17 Breakaway_Tabs, J18 Breakaway_Tabs, J19 Breakaway_Tabs, J2 AVR-ISP-6, J20 Breakaway_Tabs, J3 Breakaway_Tabs, J5 Breakaway_Tabs, J6 Breakaway_Tabs, J7 Breakaway_Tabs, J9 Breakaway_Tabs, Q1 2N7002, Q2 2N7002, SW1 SW_Push, SW2 SW_Push, U1 ATmega32U4-MU, U2 PRTR5V0U2X, U3 ATmega32U4-MU, U4 PRTR5V0U2X, Y1 16MHz, Y2 16MHz

Commit message: Update orbit-x to production copy
Parts:
- removed D63, D64, D65, D66, D67, D68, D69: SOD-123, Diodes_SMD:D_SOD-123
- removed D70, D71, D72, D73, D74: LED_3mm, locallib:LED_D3.0mm
- removed D75, D76: Schottky, Diodes_SMD:D_SOD-123
- removed G*** (x2): LOGO, locallib:Orbit
- removed G***: LOGO, locallib:ai-outline-7.6
- removed G*** (x2): LOGO, locallib:ai-ring-6mm-FancyAss
- removed G*** (x2): LOGO, locallib:ai-ring-6mm-Combined
- removed MH1, MH2: HOLE, Mounting_Holes:MountingHole_5mm
- removed MX61, MX62, MX64, MX65, MX66, MX67, MX68: MX-1U, MX_Alps_Hybrid:MX-1U
- removed MX63: MX-1.5U, MX_Alps_Hybrid:MXOnly-1.5U-Vertical
- removed MXA1, MXA2: ALPS-1.5U, MX_Alps_Hybrid:ALPS-1.5U
- removed MXE-1, MXE-2: MX-2U, MX_Alps_Hybrid:MX-2U
- removed MXE-3, MXE-4, MXE-5, MXE-6: MX-2U, MX_Alps_Hybrid:MX-2U-ReversedStabilizers
- removed Q1, Q2: 2N7002, TO_SOT_Packages_SMD:SOT-23
- removed R11, R12, R13, R14, R15, R16, R17, R18, R19, R2, R20, R21, R22, R23, R24, R26, R27, R28, R29, R3, R30, R31, R32, R34, R35, R36, R37, R38, R39, R4, R46, R47, R48, R49, R5, R50, R51, R52, R53, R54, R55, R56, R57, R58, R59, R6, R60, R61, R62, R63, R64, R65, R66, R68, R69, R7, R70, R71, R72, R73, R74, R75, R76, R77, R78, R79, R8, R80: 470, Resistors_SMD:R_0805
- removed R33, R40, R81, R82, R89, R90, R91, R92: 1k, Resistors_SMD:R_0805
- C1, C10, C11, C12, C13, C2, C3, C4, C5, C6, C7, C8, C9: footprint Capacitors_SMD:C_0603 -> Capacitor_SMD:C_0603_1608Metric; moved to F.Cu
- C14: footprint Capacitors_SMD:C_0603 -> Diode_SMD:D_SOD-123; moved to F.Cu
- D1, D2: value SOD-123 -> Schottky; footprint Diodes_SMD:D_SOD-123 -> Diode_SMD:D_SOD-123; moved to F.Cu
- D10, D11, D12, D13, D14, D15, D16, D17, D18, D19, D20, D21, D22, D23, D24, D25, D26, D27, D28, D29, D3, D30, D31, D32, D33, D34, D36, D37, D38, D39, D4, D40, D41, D42, D43, D44, D45, D46, D47, D48, D49, D5, D50, D51, D52, D53, D54, D55, D56, D57, D58, D59, D6, D60, D61, D62, D7, D8, D9: footprint Diodes_SMD:D_SOD-123 -> Diode_SMD:D_SOD-123; moved to F.Cu
- D35: value LED_3mm -> SOD-123; footprint locallib:LED_D3.0mm -> Diode_SMD:D_SOD-123
- F1, F2: footprint Fuse_Holders_and_Fuses:Fuse_SMD1206_Reflow -> Fuse:Fuse_1206_3216Metric; moved to F.Cu
- FID1, FID2, FID3: footprint Fiducials:Fiducial_1mm_Dia_2.54mm_Outer_CopperTop -> Fiducial:Fiducial_1mm_Mask3mm
- FID4, FID5, FID6: footprint Fiducials:Fiducial_1mm_Dia_2.54mm_Outer_CopperTop -> Fiducial:Fiducial_1mm_Mask3mm; moved to F.Cu
- J1, J11, J12, J2, SW1, SW2, U2, U4, USB1, USB2: moved to F.Cu
- MX34: value MX-1.5U -> MX-1U; footprint MX_Alps_Hybrid:MXOnly-1.5U-Vertical -> MX_Alps_Hybrid:MX-1U
- R10, R25, R41, R42, R43, R44, R67, R83, R84, R85, R86, R87, R88, R9: footprint Resistors_SMD:R_0805 -> Resistor_SMD:R_0603_1608Metric; moved to F.Cu
- U1, U3: footprint Housings_DFN_QFN:QFN-44-1EP_7x7mm_Pitch0.5mm -> Package_DFN_QFN:QFN-44-1EP_7x7mm_P0.5mm_EP5.15x5.15mm; moved to F.Cu
- Y1, Y2: footprint Crystals:Crystal_SMD_3225-4pin_3.2x2.5mm -> Crystal:Crystal_SMD_3225-4Pin_3.2x2.5mm; moved to F.Cu
- moved FID1 523.3 mm to (551.4, 84.4)
- moved FID6 522.4 mm to (550.9, 91.1)
- moved FID3 510.7 mm to (539.9, 97.8)
- moved D35 509.7 mm to (546.2, 73.7), turned to 0 degrees
- moved D1 498.7 mm to (546.2, 63.7), turned to 0 degrees
- moved D29 496.1 mm to (546.2, 83.8), turned to 0 degrees
- moved D15 492.9 mm to (540.5, 80.4), turned to 0 degrees
- moved D23 486.8 mm to (552.0, 77.1), turned to 0 degrees
- moved D16 474.6 mm to (540.5, 83.8), turned to 0 degrees
- moved D30 462.6 mm to (546.2, 87.1), turned to 0 degrees
- moved D3 455.9 mm to (540.5, 63.7), turned to 0 degrees
- moved D25 448.2 mm to (552.0, 80.4), turned to 0 degrees
- moved D18 442.3 mm to (546.2, 80.4), turned to 0 degrees
- moved D26 439.5 mm to (546.2, 77.1), turned to 0 degrees
- moved D31 437.2 mm to (540.5, 90.5), turned to 0 degrees
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Connections:
- D1 pad 1: ROW0 -> +5V
- D1 pad 2: Net-(D1-Pad2) -> VBUS
- D2 pad 1: ROW0 -> +5VA
- D2 pad 2: Net-(D2-Pad2) -> VDC
- D21 pad 1: ROW2 -> ROW3
- D27 pad 1: ROW3 -> Net-(D27-Pad1)
- D28 pad 1: ROW3 -> ROW4
- D33 pad 1: ROW4 -> ROW0-R
- D34 pad 1: ROW4 -> ROW0-R
- D35 pad 1: GND -> ROW0-R
- D39 pad 1: ROW0-R -> ROW1-R
- D40 pad 1: ROW0-R -> ROW1-R
- D41 pad 1: ROW0-R -> ROW1-R
- D42 pad 1: ROW0-R -> ROW1-R
- D45 pad 1: ROW1-R -> ROW2-R
- D46 pad 1: ROW1-R -> ROW2-R
- D47 pad 1: ROW1-R -> ROW2-R
- D48 pad 1: ROW1-R -> ROW2-R
- D49 pad 1: ROW1-R -> ROW2-R
- D51 pad 1: ROW2-R -> ROW3-R
- D52 pad 1: ROW2-R -> ROW3-R
- D53 pad 1: ROW2-R -> ROW3-R
- D54 pad 1: ROW2-R -> ROW3-R
- D55 pad 1: ROW2-R -> ROW3-R
- D56 pad 1: ROW2-R -> ROW3-R
- D57 pad 1: ROW3-R -> Net-(D57-Pad1)
- D58 pad 1: ROW3-R -> ROW4-R
- D59 pad 1: ROW3-R -> ROW4-R
- D60 pad 1: ROW3-R -> ROW4-R
- D61 pad 1: ROW3-R -> ROW4-R
- D62 pad 1: ROW3-R -> ROW4-R
- D8 pad 1: ROW1 -> ROW0
- MX1 pad 2: Net-(D1-Pad2) -> Net-(D3-Pad2)
- MX1 pad 3: +5V -> Net-(MX1-Pad3)
- MX10 pad 1: COL2 -> COL3
- MX10 pad 2: Net-(D10-Pad2) -> Net-(D12-Pad2)
- MX10 pad 3: +5V -> Net-(MX10-Pad3)
- MX11 pad 1: COL3 -> COL4
- MX11 pad 2: Net-(D11-Pad2) -> Net-(D13-Pad2)
- MX11 pad 3: +5V -> Net-(MX11-Pad3)
- MX12 pad 1: COL4 -> COL5
- MX12 pad 2: Net-(D12-Pad2) -> Net-(D14-Pad2)
- MX12 pad 3: +5V -> Net-(MX12-Pad3)
- MX13 pad 1: COL5 -> COL0
- MX13 pad 2: Net-(D13-Pad2) -> Net-(D15-Pad2)
- MX13 pad 3: +5V -> Net-(MX13-Pad3)
- MX14 pad 1: COL6 -> COL1
- MX14 pad 2: Net-(D14-Pad2) -> Net-(D16-Pad2)
- MX14 pad 3: +5V -> Net-(MX14-Pad3)
- MX15 pad 1: COL0 -> COL2
- MX15 pad 2: Net-(D15-Pad2) -> Net-(D17-Pad2)
- MX15 pad 3: +5V -> Net-(MX15-Pad3)
- MX16 pad 1: COL1 -> COL3
- MX16 pad 2: Net-(D16-Pad2) -> Net-(D18-Pad2)
- MX16 pad 3: +5V -> Net-(MX16-Pad3)
- MX17 pad 1: COL2 -> COL4
- MX17 pad 2: Net-(D17-Pad2) -> Net-(D19-Pad2)
- MX17 pad 3: +5V -> Net-(MX17-Pad3)
- MX18 pad 1: COL3 -> COL5
- MX18 pad 2: Net-(D18-Pad2) -> Net-(D20-Pad2)
- MX18 pad 3: +5V -> Net-(MX18-Pad3)
- MX19 pad 1: COL4 -> COL0
- MX19 pad 2: Net-(D19-Pad2) -> Net-(D21-Pad2)
- MX19 pad 3: +5V -> Net-(MX19-Pad3)
- MX2 pad 2: Net-(D2-Pad2) -> Net-(D4-Pad2)
- MX2 pad 3: +5V -> Net-(MX2-Pad3)
- MX20 pad 1: COL5 -> COL1
- MX20 pad 2: Net-(D20-Pad2) -> Net-(D22-Pad2)
- MX20 pad 3: +5V -> Net-(MX20-Pad3)
- MX21 pad 1: COL6 -> COL2
- MX21 pad 2: Net-(D21-Pad2) -> Net-(D23-Pad2)
- MX21 pad 3: +5V -> Net-(MX21-Pad3)
- MX22 pad 1: COL0 -> COL3
- MX22 pad 2: Net-(D22-Pad2) -> Net-(D24-Pad2)
- MX22 pad 3: +5V -> Net-(MX22-Pad3)
- MX23 pad 1: COL1 -> COL4
- MX23 pad 2: Net-(D23-Pad2) -> Net-(D25-Pad2)
- MX23 pad 3: +5V -> Net-(MX23-Pad3)
- MX24 pad 1: COL2 -> COL5
- MX24 pad 2: Net-(D24-Pad2) -> Net-(D26-Pad2)
- MX24 pad 3: +5V -> Net-(MX24-Pad3)
- MX25 pad 1: COL3 -> COL0
- MX25 pad 2: Net-(D25-Pad2) -> Net-(D27-Pad2)
- MX25 pad 3: +5V -> Net-(MX25-Pad3)
- MX26 pad 1: COL4 -> COL1
- MX26 pad 2: Net-(D26-Pad2) -> Net-(D28-Pad2)
- MX26 pad 3: +5V -> Net-(MX26-Pad3)
- MX27 pad 1: COL5 -> COL2
- MX27 pad 2: Net-(D27-Pad2) -> Net-(D29-Pad2)
- MX27 pad 3: +5V -> Net-(MX27-Pad3)
- MX28 pad 1: COL6 -> COL3
- MX28 pad 2: Net-(D28-Pad2) -> Net-(D30-Pad2)
- MX28 pad 3: +5V -> Net-(MX28-Pad3)
- MX29 pad 1: COL1 -> COL4
- MX29 pad 2: Net-(D29-Pad2) -> Net-(D31-Pad2)
- MX29 pad 3: +5V -> Net-(MX29-Pad3)
- MX3 pad 2: Net-(D3-Pad2) -> Net-(D5-Pad2)
- MX3 pad 3: +5V -> Net-(MX3-Pad3)
- MX30 pad 1: COL2 -> COL5
- MX30 pad 2: Net-(D30-Pad2) -> Net-(D32-Pad2)
- MX30 pad 3: +5V -> Net-(MX30-Pad3)
- MX31 pad 1: COL3 -> COL0-R
- MX31 pad 2: Net-(D31-Pad2) -> Net-(D33-Pad2)
- MX31 pad 3: +5V -> Net-(MX31-Pad3)
- MX32 pad 1: COL4 -> COL1-R
- MX32 pad 2: Net-(D32-Pad2) -> Net-(D34-Pad2)
- MX32 pad 3: +5V -> Net-(MX32-Pad3)
- MX33 pad 1: COL5 -> COL2-R
- MX33 pad 2: Net-(D33-Pad2) -> Net-(D35-Pad2)
- MX33 pad 3: +5V -> Net-(MX33-Pad3)
- MX34 pad 1: COL6 -> COL3-R
- MX34 pad 2: Net-(D34-Pad2) -> Net-(D36-Pad2)
- MX34 pad 3: +5V -> Net-(MX34-Pad3)
- MX35 pad 1: COL0-R -> COL4-R
- MX35 pad 2: Net-(D36-Pad2) -> Net-(D37-Pad2)
- MX35 pad 3: +5VA -> Net-(MX35-Pad3)
- MX36 pad 1: COL1-R -> COL5-R
- MX36 pad 2: Net-(D37-Pad2) -> Net-(D38-Pad2)
- MX36 pad 3: +5VA -> Net-(MX36-Pad3)
- MX37 pad 1: COL2-R -> COL0-R
- MX37 pad 2: Net-(D38-Pad2) -> Net-(D39-Pad2)
- MX37 pad 3: +5VA -> Net-(MX37-Pad3)
- MX38 pad 1: COL3-R -> COL1-R
- MX38 pad 2: Net-(D39-Pad2) -> Net-(D40-Pad2)
- MX38 pad 3: +5VA -> Net-(MX38-Pad3)
- MX39 pad 1: COL4-R -> COL2-R
- MX39 pad 2: Net-(D40-Pad2) -> Net-(D41-Pad2)
- MX39 pad 3: +5VA -> Net-(MX39-Pad3)
- MX4 pad 2: Net-(D4-Pad2) -> Net-(D6-Pad2)
- MX4 pad 3: +5V -> Net-(MX4-Pad3)
- MX40 pad 1: COL5-R -> COL3-R
- MX40 pad 2: Net-(D41-Pad2) -> Net-(D42-Pad2)
- MX40 pad 3: +5VA -> Net-(MX40-Pad3)
- MX41 pad 1: COL6-R -> COL4-R
- MX41 pad 2: Net-(D42-Pad2) -> Net-(D43-Pad2)
- MX41 pad 3: +5VA -> Net-(MX41-Pad3)
- MX42 pad 1: COL0-R -> COL5-R
- MX42 pad 2: Net-(D43-Pad2) -> Net-(D44-Pad2)
- MX42 pad 3: +5VA -> Net-(MX42-Pad3)
- MX43 pad 1: COL1-R -> COL0-R
- MX43 pad 2: Net-(D44-Pad2) -> Net-(D45-Pad2)
- MX43 pad 3: +5VA -> Net-(MX43-Pad3)
- MX44 pad 1: COL2-R -> COL1-R
- MX44 pad 2: Net-(D45-Pad2) -> Net-(D46-Pad2)
- MX44 pad 3: +5VA -> Net-(MX44-Pad3)
- MX45 pad 1: COL3-R -> COL2-R
- MX45 pad 2: Net-(D46-Pad2) -> Net-(D47-Pad2)
- MX45 pad 3: +5VA -> Net-(MX45-Pad3)
- MX46 pad 1: COL4-R -> COL3-R
- MX46 pad 2: Net-(D47-Pad2) -> Net-(D48-Pad2)
- MX46 pad 3: +5VA -> Net-(MX46-Pad3)
- MX47 pad 1: COL5-R -> COL4-R
- MX47 pad 2: Net-(D48-Pad2) -> Net-(D49-Pad2)
- MX47 pad 3: +5VA -> Net-(MX47-Pad3)
- MX48 pad 1: COL6-R -> COL5-R
- MX48 pad 2: Net-(D49-Pad2) -> Net-(D50-Pad2)
- MX48 pad 3: +5VA -> Net-(MX48-Pad3)
- MX49 pad 2: Net-(D50-Pad2) -> Net-(D51-Pad2)
- MX49 pad 3: +5VA -> Net-(MX49-Pad3)
- MX5 pad 2: Net-(D5-Pad2) -> Net-(D7-Pad2)
- MX5 pad 3: +5V -> Net-(MX5-Pad3)
- MX50 pad 2: Net-(D51-Pad2) -> Net-(D52-Pad2)
- MX50 pad 3: +5VA -> Net-(MX50-Pad3)
- MX51 pad 2: Net-(D52-Pad2) -> Net-(D53-Pad2)
- MX51 pad 3: +5VA -> Net-(MX51-Pad3)
- MX52 pad 2: Net-(D53-Pad2) -> Net-(D54-Pad2)
- MX52 pad 3: +5VA -> Net-(MX52-Pad3)
- MX53 pad 2: Net-(D54-Pad2) -> Net-(D55-Pad2)
- MX53 pad 3: +5VA -> Net-(MX53-Pad3)
- MX54 pad 2: Net-(D55-Pad2) -> Net-(D56-Pad2)
- MX54 pad 3: +5VA -> Net-(MX54-Pad3)
- MX55 pad 1: COL6-R -> COL0-R
- MX55 pad 2: Net-(D56-Pad2) -> Net-(D57-Pad2)
- MX55 pad 3: +5VA -> Net-(MX55-Pad3)
- MX56 pad 1: COL0-R -> COL1-R
- MX56 pad 2: Net-(D57-Pad2) -> Net-(D58-Pad2)
- MX56 pad 3: +5VA -> Net-(MX56-Pad3)
- MX57 pad 1: COL1-R -> COL2-R
- MX57 pad 2: Net-(D58-Pad2) -> Net-(D59-Pad2)
- MX57 pad 3: +5VA -> Net-(MX57-Pad3)
- MX58 pad 1: COL2-R -> COL3-R
- MX58 pad 2: Net-(D59-Pad2) -> Net-(D60-Pad2)
- MX58 pad 3: +5VA -> Net-(MX58-Pad3)
- MX59 pad 1: COL3-R -> COL4-R
- MX59 pad 2: Net-(D60-Pad2) -> Net-(D61-Pad2)
- MX59 pad 3: +5VA -> Net-(MX59-Pad3)
- MX6 pad 2: Net-(D6-Pad2) -> Net-(D8-Pad2)
- MX6 pad 3: +5V -> Net-(MX6-Pad3)
- MX60 pad 1: COL4-R -> COL5-R
- MX60 pad 2: Net-(D61-Pad2) -> Net-(D62-Pad2)
- MX60 pad 3: +5VA -> Net-(MX60-Pad3)
- MX7 pad 1: COL6 -> COL0
- MX7 pad 2: Net-(D7-Pad2) -> Net-(D9-Pad2)
- MX7 pad 3: +5V -> Net-(MX7-Pad3)
- MX8 pad 1: COL0 -> COL1
- MX8 pad 2: Net-(D8-Pad2) -> Net-(D10-Pad2)
- MX8 pad 3: +5V -> Net-(MX8-Pad3)
- MX9 pad 1: COL1 -> COL2
- MX9 pad 2: Net-(D9-Pad2) -> Net-(D11-Pad2)
- MX9 pad 3: +5V -> Net-(MX9-Pad3)
Routing:
- net +5V: track 980.7 -> 0.00 mm, vias 14 -> 0
- net +5VA: track 945.4 -> 0.00 mm, vias 13 -> 0
- net LEDGND-R: track 681.7 -> 0.00 mm, vias 19 -> 0
- net LEDGND: track 666.3 -> 0.00 mm, vias 17 -> 0
- net GND: track 540.0 -> 0.00 mm, vias 5 -> 0
- net GNDA: track 510.4 -> 0.00 mm, vias 6 -> 0
- net ROW0-R: track 205.8 -> 0.00 mm, vias 4 -> 0
- net ROW0: track 196.3 -> 0.00 mm, vias 4 -> 0
- net ROW1-R: track 177.0 -> 0.00 mm, vias 4 -> 0
- net ROW1: track 173.1 -> 0.00 mm, vias 4 -> 0
- net COL0: track 167.9 -> 0.00 mm
- net COL1: track 163.0 -> 0.00 mm
- net ROW2-R: track 159.8 -> 0.00 mm, vias 4 -> 0
- net ROW2: track 155.7 -> 0.00 mm, vias 4 -> 0
- net COL5-R: track 150.8 -> 0.00 mm
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- removed copper zone on B.Cu, net GND
- removed copper zone on B.Cu, net GNDA
Other:
- board outline removed
- board text removed: "L"
- board text removed: "Orbit PCB R2.2 by ai03"
- board text removed: "Orbit PCB Revision 2.2 20181211"
- board text removed: "R"
- board text removed: "RESET"
